File: nrfstick.kicad_sch (KiCad schematic)
At the start: 28 parts, among them J1 USB_A, J2 programming conn, SW4 SW_Push, U3 APX803L20-27SR-7, U4 CP2102C-Axx-xQFN24, U5 BM15C, Y1 32.768kHz

Commit message: Start AB changes - add RTS/CTS
squash
Parts:
- J2: now fitted
Connections:
- net UART_nRF_RTS: now reaches U5.G8 (P1.08)
- net UART_nRF_RTS: now also U4.18 (~{CTS})
- net UART_nRF_CTS: now reaches U5.G9 (P1.07/AIN3)
- net UART_nRF_CTS: now also U4.19 (~{RTS})
- no-connect marks 32 -> 28
Changed lines of the file:
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@@
 	)
 	(no_connect
-		(at 273.05 83.82)
-	)
-	(no_connect
 		(at 252.73 186.69)
 	)
@@
 	)
 	(no_connect
-		(at 273.05 81.28)
-	)
-	(no_connect
 		(at 252.73 171.45)
 	)
 	(no_connect
-		(at 196.85 193.04)
-	)
-	(no_connect
-		(at 196.85 190.5)
-	)
-	(no_connect
 		(at 252.73 173.99)
 	)
@@
 	(wire
 		(pts
+			(xy 195.58 185.42) (xy 196.85 185.42)
+		)
+		(stroke
+			(width 0)
+			(type default)
+		)
+	)
+	(wire
+		(pts
 			(xy 199.39 86.36) (xy 213.36 86.36)
 		)
@@
 	(wire
 		(pts
-			(xy 273.05 76.2) (xy 276.86 76.2)
-		)
-		(stroke
-			(width 0)
-			(type default)
-		)
-	)
-	(wire
-		(pts
 			(xy 191.77 135.89) (xy 191.77 129.54)
 		)
@@
 	(wire
 		(pts
-			(xy 181.61 187.96) (xy 196.85 187.96)
+			(xy 195.58 187.96) (xy 196.85 187.96)
 		)
 		(stroke
@@
 	(wire
 		(pts
-			(xy 181.61 198.12) (xy 196.85 198.12)
+			(xy 195.58 190.5) (xy 196.85 190.5)
 		)
 		(stroke
@@
 	(wire
 		(pts
-			(xy 246.38 76.2) (xy 247.65 76.2)
+			(xy 181.61 198.12) (xy 196.85 198.12)
 		)
 		(stroke
@@
 	(wire
 		(pts
-			(xy 181.61 185.42) (xy 196.85 185.42)
+			(xy 246.38 76.2) (xy 247.65 76.2)
 		)
 		(stroke
@@
 	(wire
 		(pts
-			(xy 273.05 78.74) (xy 276.86 78.74)
-		)
-		(stroke
-			(width 0)
-			(type default)
-		)
-	)
-	(wire
-		(pts
 			(xy 137.16 228.6) (xy 137.16 229.87)
 		)
@@
 	(wire
 		(pts
+			(xy 195.58 193.04) (xy 196.85 193.04)
+		)
+		(stroke
+			(width 0)
+			(type default)
+		)
+	)
+	(wire
+		(pts
 			(xy 223.52 228.6) (xy 223.52 227.33)
 		)
@@
 	)
 	(label "UART_nRF_TX"
-		(at 181.61 185.42 0)
+		(at 195.58 185.42 180)
 		(effects
 			(font
 				(size 1.27 1.27)
 			)
-			(justify left bottom)
+			(justify right bottom)
 		)
 	)
@@
 		)
 	)
+	(label "UART_nRF_RTS"
+		(at 195.58 193.04 180)
+		(effects
+			(font
+				(size 1.27 1.27)
+			)
+			(justify right bottom)
+		)
+	)
+	(label "UART_nRF_CTS"
+		(at 273.05 81.28 0)
+		(effects
+			(font
+				(size 1.27 1.27)
+			)
+			(justify left bottom)
+		)
+	)
 	(label "LED_BLUE"
 		(at 137.16 207.01 0)
@@
 	)
 	(label "UART_nRF_RX"
-		(at 181.61 187.96 0)
+		(at 195.58 187.96 180)
 		(effects
 			(font
 				(size 1.27 1.27)
 			)
-			(justify left bottom)
+			(justify right bottom)
 		)
 	)
@@
 		)
 	)
+	(label "UART_nRF_RTS"
+		(at 273.05 83.82 0)
+		(effects
+			(font
+				(size 1.27 1.27)
+			)
+			(justify left bottom)
+		)
+	)
+	(label "UART_nRF_CTS"
+		(at 195.58 190.5 180)
+		(effects
+			(font
+				(size 1.27 1.27)
+			)
+			(justify right bottom)
+		)
+	)
 	(label "UART_nRF_RX"
-		(at 276.86 76.2 0)
+		(at 273.05 76.2 0)
 		(effects
 			(font
@@
 	)
 	(label "UART_nRF_TX"
-		(at 276.86 78.74 0)
+		(at 273.05 78.74 0)
 		(effects
 			(font
@@
 		(on_board yes)
 		(in_pos_files yes)
-		(dnp yes)
+		(dnp no)
 		(property "Reference" "J2"
 			(at 263.652 137.922 0)

Commit message: Replace SW4 with Alps SKRPABE010 and save revised PCB layout
Parts:
- SW4: value SW_Push -> SKRPABE010; footprint footprint:SW_STU-057A23AC_8127_2.25N -> footprint:SW_Push_Alps_SKRPABE010; MFR Mitsumi -> Alps Alpine; MFR_PN R-668127 -> SKRPABE010
Changed lines of the file:
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@@
 			)
 		)
-		(property "Value" "SW_Push"
+		(property "Value" "SKRPABE010"
 			(at 266.7 219.71 0)
 			(hide yes)
@@
 			)
 		)
-		(property "Footprint" "footprint:SW_STU-057A23AC_8127_2.25N"
+		(property "Footprint" "footprint:SW_Push_Alps_SKRPABE010"
 			(at 266.7 219.71 0)
 			(hide yes)
@@
 			)
 		)
-		(property "Datasheet" ""
+		(property "Datasheet" "https://tech.alpsalpine.com/e/products/detail/SKRPABE010/"
 			(at 266.7 219.71 0)
 			(hide yes)
@@
 			)
 		)
-		(property "Description" ""
+		(property "Description" "SMD tactile switch, NO, 4.2x3.2mm, 2.5mm high, 1.57N"
 			(at 261.62 219.71 0)
 			(hide yes)
@@
 			)
 		)
-		(property "MFR" "Mitsumi"
+		(property "MFR" "Alps Alpine"
 			(at 261.62 219.71 0)
 			(hide yes)
@@
 			)
 		)
-		(property "MFR_PN" "R-668127 "
+		(property "MFR_PN" "SKRPABE010"
 			(at 261.62 219.71 0)
 			(hide yes)

Commit message: panel layout using kikit, not routed
Parts:
- added J3: IO00, footprint:Conn_Pads_1x04_P2.00mm_D1.00mm, symbol Connector:Conn_01x04_Pin
- added J4: Reset, footprint:Conn_Pads_2x01_P2.00mm_D1.00mm, symbol Connector:Conn_01x02_Pin
- added J6: UART2, footprint:Conn_Pads_1x04_P2.00mm_D1.00mm, symbol Connector:Conn_01x04_Pin
- renumbered SW4 to SW1
Connections:
- net GND: now also J4.1 (Pin_1)
- net at C20.2, R17.2, R29.2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: now also J4.2 (Pin_2)
- net at U5.H9 (P2.00): now also J6.1 (Pin_1)
- net at U5.J2 (P0.03): now also J3.1 (Pin_1)
- net at U5.J4 (P0.00): now also J3.4 (Pin_4)
- net at U5.J7 (P2.03): now also J6.4 (Pin_4)
- net at U5.J8 (P2.02): now also J6.3 (Pin_3)
- net at U5.J9 (P2.01): now also J6.2 (Pin_2)
- net at U5.K2 (P0.02): now also J3.2 (Pin_2)
- net at U5.K4 (P0.01): now also J3.3 (Pin_3)
- no-connect marks 28 -> 20

Commit message: panelize, new usb connector
Parts:
- J1: footprint footprint:connector-USB-A-male-smd-Molex-480372100 -> footprint:USB_A_AdamTech_USB-AP-S-RA-SMT; MFR Molex -> Adam Tech; MFR_PN 480372100 -> USB-AP-S-RA-SMT
Changed lines of the file:
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@@
 			)
 		)
-		(property "Footprint" "footprint:connector-USB-A-male-smd-Molex-480372100"
+		(property "Footprint" "footprint:USB_A_AdamTech_USB-AP-S-RA-SMT"
 			(at 152.4 73.914 0)
 			(hide yes)
@@
 			)
 		)
-		(property "Datasheet" ""
+		(property "Datasheet" "data/usb-ap-s-ra-smt-data-sheet.pdf"
 			(at 153.67 91.44 0)
 			(hide yes)
@@
 			)
 		)
-		(property "MFR" "Molex"
+		(property "MFR" "Adam Tech"
 			(at 149.86 90.17 0)
 			(hide yes)
@@
 			)
 		)
-		(property "MFR_PN" "480372100"
+		(property "MFR_PN" "USB-AP-S-RA-SMT"
 			(at 149.86 90.17 0)
 			(hide yes)
